File: digitalSystemBoard/Header_and_Mounting.sch (KiCad schematic (older format))
At the start: 30 parts, among them J10 Conn_02x03_Odd_Even, J11 Conn_02x03_Odd_Even, J2 Conn_02x04_Odd_Even, J3 Conn_02x04_Odd_Even, J4 Conn_02x08_Odd_Even, J5 Conn_02x07_Odd_Even, J6 Conn_02x07_Odd_Even, J7 Conn_02x08_Odd_Even, J8 Conn_02x03_Odd_Even, J9 Conn_02x03_Odd_Even

Commit message: Generate BOM, Gerber and CPL file
Parts:
- R74, R75, R76, R77, R78, R79, R80, R81: LCSC C98220 -> C105579
Changed lines of the file:
@@
 F 2 "Resistor_SMD:R_0603_1608Metric" V 7810 2000 50  0001 C CNN
 F 3 "~" H 7880 2000 50  0001 C CNN
-F 4 "C98220" V 7880 2000 50  0001 C CNN "LCSC"
+F 4 "C105579" V 7880 2000 50  0001 C CNN "LCSC"
 	1    7880 2000
 	0    1    1    0
@@
 F 2 "Resistor_SMD:R_0603_1608Metric" V 7810 2170 50  0001 C CNN
 F 3 "~" H 7880 2170 50  0001 C CNN
-F 4 "C98220" V 7880 2170 50  0001 C CNN "LCSC"
+F 4 "C105579" V 7880 2170 50  0001 C CNN "LCSC"
 	1    7880 2170
 	0    1    1    0
@@
 F 2 "Resistor_SMD:R_0603_1608Metric" V 7810 2340 50  0001 C CNN
 F 3 "~" H 7880 2340 50  0001 C CNN
-F 4 "C98220" V 7880 2340 50  0001 C CNN "LCSC"
+F 4 "C105579" V 7880 2340 50  0001 C CNN "LCSC"
 	1    7880 2340
 	0    1    1    0
@@
 F 2 "Resistor_SMD:R_0603_1608Metric" V 7810 2510 50  0001 C CNN
 F 3 "~" H 7880 2510 50  0001 C CNN
-F 4 "C98220" V 7880 2510 50  0001 C CNN "LCSC"
+F 4 "C105579" V 7880 2510 50  0001 C CNN "LCSC"
 	1    7880 2510
 	0    1    1    0
@@
 F 2 "Resistor_SMD:R_0603_1608Metric" V 7810 2680 50  0001 C CNN
 F 3 "~" H 7880 2680 50  0001 C CNN
-F 4 "C98220" V 7880 2680 50  0001 C CNN "LCSC"
+F 4 "C105579" V 7880 2680 50  0001 C CNN "LCSC"
 	1    7880 2680
 	0    1    1    0
@@
 F 2 "Resistor_SMD:R_0603_1608Metric" V 7810 2850 50  0001 C CNN
 F 3 "~" H 7880 2850 50  0001 C CNN
-F 4 "C98220" V 7880 2850 50  0001 C CNN "LCSC"
+F 4 "C105579" V 7880 2850 50  0001 C CNN "LCSC"
 	1    7880 2850
 	0    1    1    0
@@
 F 2 "Resistor_SMD:R_0603_1608Metric" V 7810 3030 50  0001 C CNN
 F 3 "~" H 7880 3030 50  0001 C CNN
-F 4 "C98220" V 7880 3030 50  0001 C CNN "LCSC"
+F 4 "C105579" V 7880 3030 50  0001 C CNN "LCSC"
 	1    7880 3030
 	0    1    1    0
@@
 F 2 "Resistor_SMD:R_0603_1608Metric" V 7810 3200 50  0001 C CNN
 F 3 "~" H 7880 3200 50  0001 C CNN
-F 4 "C98220" V 7880 3200 50  0001 C CNN "LCSC"
+F 4 "C105579" V 7880 3200 50  0001 C CNN "LCSC"
 	1    7880 3200
 	0    1    1    0
