File: digitalSystemBoard/MCU.sch (KiCad schematic (older format))
At the start: 31 parts, among them J1 USB-B, J12 Conn_01x10_Female, J13 Conn_01x10_Female, J14 Conn_01x10_Female, J15 Conn_01x10_Female, SW9 ButtonFirst, U10 74HC165, U11 74HC595, U7 ICSP, U8 74HC165, U9 74HC595

Commit message: Generate BOM, Gerber and CPL file
Parts:
- U10, U8: LCSC C7742 -> C5613
Changed lines of the file:
@@
 F 2 "Package_SO:SOIC-16_3.9x9.9mm_P1.27mm" H 6290 3590 50  0001 C CNN
 F 3 "http://www.ti.com/lit/gpn/sn74LS165" H 6290 3590 50  0001 C CNN
-F 4 "C7742" H 6290 3590 50  0001 C CNN "LCSC"
+F 4 "C5613" H 6290 3590 50  0001 C CNN "LCSC"
 	1    6290 3590
 	1    0    0    -1
@@
 F 2 "Package_SO:SOIC-16_3.9x9.9mm_P1.27mm" H 9290 3590 50  0001 C CNN
 F 3 "http://www.ti.com/lit/gpn/sn74LS165" H 9290 3590 50  0001 C CNN
-F 4 "C7742" H 9290 3590 50  0001 C CNN "LCSC"
+F 4 "C5613" H 9290 3590 50  0001 C CNN "LCSC"
 	1    9290 3590
 	1    0    0    -1
