File: digitalSystemBoard/SWITCH_AND_BUTTON.sch (KiCad schematic (older format))
At the start: 65 parts, among them Q10 BC847, Q11 BC847, Q12 BC847, Q13 BC847, Q14 BC847, Q15 BC847, Q8 BC847, Q9 BC847, SW1 IO_Switch, SW2 IO_Switch, SW3 IO_Switch, SW4 IO_Switch, SW5 IO_Switch, SW6 IO_Switch, SW7 IO_Switch, SW8 IO_Switch, U4 74LS04, U5 Potentiometer

Commit message: Generate BOM, Gerber and CPL file
Parts:
- U4: LCSC C6796 -> C510568
Changed lines of the file:
@@
 F 2 "Package_SO:SOIC-14_3.9x8.7mm_P1.27mm" H 3540 5550 50  0001 C CNN
 F 3 "http://www.ti.com/lit/gpn/sn74LS04" H 3540 5550 50  0001 C CNN
-F 4 "C6796" H 3540 5550 50  0001 C CNN "LCSC"
+F 4 "C510568" H 3540 5550 50  0001 C CNN "LCSC"
 	1    3540 5550
 	1    0    0    -1
@@
 F 2 "Package_SO:SOIC-14_3.9x8.7mm_P1.27mm" H 6830 5070 50  0001 C CNN
 F 3 "http://www.ti.com/lit/gpn/sn74LS04" H 6830 5070 50  0001 C CNN
-F 4 "C6796" H 6830 5070 50  0001 C CNN "LCSC"
+F 4 "C510568" H 6830 5070 50  0001 C CNN "LCSC"
 	7    6830 5070
 	1    0    0    -1
